Commit message: Minor

File: urdf/ur_macro.xacro (robot description, xacro)
@@ -350,5 +350,5 @@
       <parent link="${prefix}wrist_3_link" />
       <child link="${prefix}flange" />
-      <origin xyz="0 0 0.1" rpy="0 ${-pi/2.0} ${-pi/2.0}" />
+      <origin xyz="0 0 0.05" rpy="0 ${-pi/2.0} ${-pi/2.0}" />
     </joint>
     <!-- ROS-Industrial 'tool0' frame - all-zeros tool frame -->
@@ -360,4 +360,10 @@
       <child link="${prefix}tool0"/>
     </joint>
+    <link name="${prefix}camera"/>
+    <joint name="${prefix}flange-camera" type="fixed">
+      <origin xyz="0 0.0141 -0.02925" rpy="${pi} 0 ${pi/2}"/>
+      <parent link="${prefix}flange"/>
+      <child link="${prefix}camera"/>
+    </joint>
   </xacro:macro>
 </robot>
